Commit message: Reduce sensor rate

File: master3_description/urdf/yahboomcar_X3.urdf.xacro (robot description, xacro)
@@ -293,4 +293,10 @@
     <xacro:fixed_joint name="camera_joint" parent="base_link" child="camera_link"
         xyz="0.057105 1.7948E-05 0.03755" rpy="0 0 0" />
+        <joint name="camera_optical_joint" type="fixed">
+            <origin xyz="0 0 0" rpy="${-pi/2} 0 ${-pi/2}" />
+            <parent link="camera_link" />
+            <child link="camera_link_optical" />
+        </joint>
+        <link name="camera_link_optical"></link>
     <xacro:if value="${mecanum}">
         <gazebo>
@@ -515,7 +521,7 @@
         <sensor type="camera" name="camera_orbbec_astra_color">
             <always_on>true</always_on>
-            <update_rate>30.0</update_rate>
+            <update_rate>10.0</update_rate>
             <topic>/color/image_raw</topic>
-            <visualize>false</visualize>
+            <visualize>true</visualize>
             <gz_frame_id>camera_link</gz_frame_id>
             <horizontal_fov>${60.0/180.0*pi}</horizontal_fov>
@@ -535,4 +541,5 @@
             <visualize>true</visualize>
             <gz_frame_id>camera_link</gz_frame_id>
+            <!-- <gz_frame_id>camera_link_optical</gz_frame_id> -->
             <camera>
                 <horizontal_fov>${60.0/180.0*pi}</horizontal_fov>
